File: cm108b-eval.sch (KiCad schematic (older format))
At the start: 42 parts, among them IC1 CM108B, J1 SPRK, J2 MIC, J3 RADIO_DATA, SW1 MUTE_REC, SW2 MUTE_PLAY, SW3 VOL_DN, SW4 VOL_UP

Commit message: Completed BOM
Parts:
- C1: value 10uF -> 10μF; Price (none) -> 0.29; Vendor (none) -> Mouser; Vendor Part # (none) -> 791-1210F106Z100CT
- C10: value 104 -> 100nF; Price (none) -> 0.37; Vendor (none) -> Mouser; Vendor Part # (none) -> 80-C1210C104K5RAUTO
- C11: value 1uF -> 1μF; Price (none) -> 0.13; Vendor (none) -> Mouser; Vendor Part # (none) -> 791-1210B105M101CT
- C14, C15, C7, C9: value 4.7uF -> 4.7μF; Price (none) -> 0.35; Vendor (none) -> Mouser; Vendor Part # (none) -> 963-EMK325B7475MN-T
- C3, C4: Price (none) -> 0.28; Vendor (none) -> Mouser; Vendor Part # (none) -> 80-C1210C101K3HACTU
- C50, C51: value 470uF -> 470μF; Price (none) -> 1.3; Vendor (none) -> Mouser
- C6, C8: Price (none) -> 0.37; Vendor (none) -> Mouser; Vendor Part # (none) -> 80-C1210C104K5RAUTO
- D1, D2, D3: footprint LED_SMD:LED_1210_3225Metric -> LED_SMD:LED_0603_1608Metric; Price (none) -> 0.15; Vendor (none) -> Mouser; Vendor Part # (none) -> 710-150060RS75000
- IC1: Price (none) -> 1.64; Vendor (none) -> Symmetry; Vendor Part # (none) -> CM108B
- J1: value SPRK -> SPKR; Price (none) -> 1.26; Vendor (none) -> Mouser
- J2: Price (none) -> 1.26; Vendor (none) -> Mouser
- J3: Price (none) -> 0.35; Vendor (none) -> Mouser; Vendor Part # (none) -> 485-4389
- JP1, JP3, JP4: Price (none) -> 0.1; Vendor (none) -> Mouser; Vendor Part # (none) -> 649-1012937890301BLF
- JP2: Price (none) -> 0.95; Vendor (none) -> Mouser; Vendor Part # (none) -> 538-47346-0001
- L1, L2: Price (none) -> 0.92; Vendor (none) -> Mouser; Vendor Part # (none) -> 673-PE1210CCMC161STS
- R1, R2: Price (none) -> 0.17; Vendor (none) -> Mouser; Vendor Part # (none) -> 667-ERJ-14YJ220U
- R10: Price (none) -> 0.2; Vendor (none) -> Mouser; Vendor Part # (none) -> 660-RK73H2ETTD2201F
- R11, R12, R7: value 330 -> 330Ω; Price (none) -> 0.13; Vendor (none) -> Mouser; Vendor Part # (none) -> 279-CRGCQ1210J330R
- R13: Price (none) -> 0.16; Vendor (none) -> Mouser; Vendor Part # (none) -> 603-RC1210FR-071K2L
- R3: Price (none) -> 0.14; Vendor (none) -> Mouser; Vendor Part # (none) -> 660-RK73Z2ETTD
- R4: Price (none) -> 0.14; Vendor (none) -> Mouser; Vendor Part # (none) -> 661-RK73Z2ETTD
- R5: Price (none) -> 0.14; Vendor (none) -> Mouser; Vendor Part # (none) -> 662-RK73Z2ETTD
- R6: Price (none) -> 0.14; Vendor (none) -> Mouser; Vendor Part # (none) -> 663-RK73Z2ETTD
- SW1, SW2, SW3, SW4: Price (none) -> 0.58; Vendor (none) -> Mouser; Vendor Part # (none) -> 653-B3FS-1002P
- TP1: Price (none) -> 0; Vendor (none) -> -; Vendor Part # (none) -> -

Commit message: Move inductor to USB cable shield
Having it on the cable's ground pin just doesn't make sense to me.
Connections:
- net GND: now also JP2.4 (GND), L2.1; no longer JP2.5 (Shield), L2.2
- new net: JP2.5 (Shield), L2.2
Other:
- moved on the sheet: L2
Changed lines of the file:
@@
-$EndComp
-$Comp
-L Connector:USB_A JP2
-U 1 1 6057963A
-P 1350 2850
-F 0 "JP2" H 1407 3317 50  0000 C CNN
-F 1 "USB_A" H 1407 3226 50  0000 C CNN
-F 2 "Connector_USB:USB_Micro-B_Molex_47346-0001" H 1500 2800 50  0001 C CNN
-F 3 "https://www.mouser.com/datasheet/2/276/0473460001_IO_CONNECTORS-229243.pdf" H 1500 2800 50  0001 C CNN
-F 4 "0.95" H 1407 3417 50  0001 C CNN "Price"
-F 5 "538-47346-0001" H 1407 3417 50  0001 C CNN "Vendor Part #"
-F 6 "Mouser" H 1407 3417 50  0001 C CNN "Vendor"
-	1    1350 2850
-	1    0    0    -1
 $EndComp
 $Comp
@@
 F 3 "" H 4900 5500 50  0001 C CNN
 	1    4900 5500
-	1    0    0    -1
-$EndComp
-$Comp
-L power:GND #PWR0102
-U 1 1 6058A2AB
-P 1350 3600
-F 0 "#PWR0102" H 1350 3350 50  0001 C CNN
-F 1 "GND" H 1355 3427 50  0001 C CNN
-F 2 "" H 1350 3600 50  0001 C CNN
-F 3 "" H 1350 3600 50  0001 C CNN
-	1    1350 3600
 	1    0    0    -1
 $EndComp
@@
 L Device:L_Core_Ferrite L2
 U 1 1 6059FDC7
-P 1350 3400
-F 0 "L2" H 1438 3446 50  0000 L CNN
-F 1 "L" H 1438 3355 50  0000 L CNN
-F 2 "Inductor_SMD:L_1210_3225Metric" H 1350 3400 50  0001 C CNN
-F 3 "https://www.mouser.com/datasheet/2/336/W719-1480588.pdf" H 1350 3400 50  0001 C CNN
-F 4 "0.92" H 1438 3546 50  0001 C CNN "Price"
-F 5 "673-PE1210CCMC161STS" H 1438 3546 50  0001 C CNN "Vendor Part #"
-F 6 "Mouser" H 1438 3546 50  0001 C CNN "Vendor"
-	1    1350 3400
-	1    0    0    -1
+P 1200 3450
+F 0 "L2" H 1288 3496 50  0000 L CNN
+F 1 "L" H 1288 3405 50  0000 L CNN
+F 2 "Inductor_SMD:L_1210_3225Metric" H 1200 3450 50  0001 C CNN
+F 3 "https://www.mouser.com/datasheet/2/336/W719-1480588.pdf" H 1200 3450 50  0001 C CNN
+F 4 "0.92" H 1288 3596 50  0001 C CNN "Price"
+F 5 "673-PE1210CCMC161STS" H 1288 3596 50  0001 C CNN "Vendor Part #"
+F 6 "Mouser" H 1288 3596 50  0001 C CNN "Vendor"
+	1    1200 3450
+	-1   0    0    1
 $EndComp
 $Comp
@@
 	2000 2850 2300 2850
 Wire Wire Line
-	1350 3600 1350 3550
-Wire Wire Line
 	1850 3600 1850 3350
 Wire Wire Line
 	2000 3600 2000 3350
-Wire Wire Line
-	1250 3250 1250 3400
-Wire Wire Line
-	1250 3400 1200 3400
-Wire Wire Line
-	1200 3400 1200 3600
 Wire Wire Line
 	9300 5150 9400 5150
@@
 NoConn ~ 4050 5050
 NoConn ~ 4050 5150
+$Comp
+L power:GND #PWR?
+U 1 1 605F61ED
+P 1350 3600
+F 0 "#PWR?" H 1350 3350 50  0001 C CNN
+F 1 "GND" H 1355 3427 50  0001 C CNN
+F 2 "" H 1350 3600 50  0001 C CNN
+F 3 "" H 1350 3600 50  0001 C CNN
+	1    1350 3600
+	1    0    0    -1
+$EndComp
+$Comp
+L Connector:USB_A JP2
+U 1 1 6057963A
+P 1350 2850
+F 0 "JP2" H 1407 3317 50  0000 C CNN
+F 1 "USB_A" H 1407 3226 50  0000 C CNN
+F 2 "Connector_USB:USB_Micro-B_Molex_47346-0001" H 1500 2800 50  0001 C CNN
+F 3 "https://www.mouser.com/datasheet/2/276/0473460001_IO_CONNECTORS-229243.pdf" H 1500 2800 50  0001 C CNN
+F 4 "0.95" H 1407 3417 50  0001 C CNN "Price"
+F 5 "538-47346-0001" H 1407 3417 50  0001 C CNN "Vendor Part #"
+F 6 "Mouser" H 1407 3417 50  0001 C CNN "Vendor"
+	1    1350 2850
+	1    0    0    -1
+$EndComp
+Wire Wire Line
+	1350 3250 1350 3600
+Wire Wire Line
+	1250 3250 1250 3300
+Wire Wire Line
+	1250 3300 1200 3300
 $EndSCHEMATC
