File: cm108b-eval.sch (KiCad schematic (older format))
At the start: 44 parts, among them IC1 CM108B, J1 SPKR, J2 MIC, J3 RADIO_DATA, SW1 MUTE_REC, SW2 MUTE_PLAY, SW3 VOL_DN, SW4 VOL_UP

Commit message: Incorporate learnings from first physical prototype
* Button footprint pad numberings are wrong for symbol, so they were always pressed
* Turn J3 for solderability
Parts:
- SW1, SW2, SW3, SW4: footprint Button_Switch_SMD:SW_SPST_Omron_B3FS-100xP -> Omron:SW_SPST_Omron_B3FS-100xP
Changed lines of the file:
@@
 Sheet 1 1
 Title "CM108B Evaluation Board"
-Date "2021-04-14"
+Date "2021-04-18"
 Rev "4"
 Comp "Chris Keller"
@@
 F 0 "SW1" H 9100 5435 50  0000 C CNN
 F 1 "MUTE_REC" H 9100 5344 50  0000 C CNN
-F 2 "Button_Switch_SMD:SW_SPST_Omron_B3FS-100xP" H 9100 5350 50  0001 C CNN
+F 2 "Omron:SW_SPST_Omron_B3FS-100xP" H 9100 5350 50  0001 C CNN
 F 3 "https://www.mouser.com/datasheet/2/307/omron_B3FS-1189765.pdf" H 9100 5350 50  0001 C CNN
 F 4 "0.58" H 9100 5535 50  0001 C CNN "Price"
@@
 F 0 "SW2" H 9100 5785 50  0000 C CNN
 F 1 "MUTE_PLAY" H 9100 5694 50  0000 C CNN
-F 2 "Button_Switch_SMD:SW_SPST_Omron_B3FS-100xP" H 9100 5700 50  0001 C CNN
+F 2 "Omron:SW_SPST_Omron_B3FS-100xP" H 9100 5700 50  0001 C CNN
 F 3 "https://www.mouser.com/datasheet/2/307/omron_B3FS-1189765.pdf" H 9100 5700 50  0001 C CNN
 F 4 "0.58" H 9100 5885 50  0001 C CNN "Price"
@@
 F 0 "SW3" H 9100 6135 50  0000 C CNN
 F 1 "VOL_DN" H 9100 6044 50  0000 C CNN
-F 2 "Button_Switch_SMD:SW_SPST_Omron_B3FS-100xP" H 9100 6050 50  0001 C CNN
+F 2 "Omron:SW_SPST_Omron_B3FS-100xP" H 9100 6050 50  0001 C CNN
 F 3 "https://www.mouser.com/datasheet/2/307/omron_B3FS-1189765.pdf" H 9100 6050 50  0001 C CNN
 F 4 "0.58" H 9100 6235 50  0001 C CNN "Price"
@@
 F 0 "SW4" H 9100 6485 50  0000 C CNN
 F 1 "VOL_UP" H 9100 6394 50  0000 C CNN
-F 2 "Button_Switch_SMD:SW_SPST_Omron_B3FS-100xP" H 9100 6400 50  0001 C CNN
+F 2 "Omron:SW_SPST_Omron_B3FS-100xP" H 9100 6400 50  0001 C CNN
 F 3 "https://www.mouser.com/datasheet/2/307/omron_B3FS-1189765.pdf" H 9100 6400 50  0001 C CNN
 F 4 "0.58" H 9100 6585 50  0001 C CNN "Price"
